File: adapter/adapter.kicad_sch (KiCad schematic)
At the start: 28 parts, among them J10 Ribbon, J11 Ribbon, J12 Ribbon, J9 Ribbon, Q1 Q_NMOS_GSD, Q2 Q_NMOS_GSD, Q3 Q_NMOS_GSD, Q4 Q_NMOS_GSD, SW1 SW_SPST, SW2 SW_SPST, SW3 SW_SPDT, SW4 SW_SPDT, U1 xiao-ble, U2 xiao-ble, U3 AP9101CK6, U4 AP9101CK6

Commit message: Fix the schematic info, add a schematic as pdf
I like to read schematics by not having to download
and open with KiCAD, so seems reasonable to do that
with my project.
Other:
- company: BastardKB x KarlK90 -> zemm
- title: Elite-C holder -> XIAO BLE AAA Adapter
Changed lines of the file:
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@@
   (paper "A4")
   (title_block
-    (title "Elite-C holder")
-    (date "2022-02-13")
-    (rev "2.0")
-    (company "BastardKB x KarlK90")
+    (title "XIAO BLE AAA Adapter")
+    (date "2024-02-25")
+    (rev "0.1")
+    (company "zemm")
     (comment 1 "Licensed under CERN-OHL-W v2")
+    (comment 2 "Based on the Elite-C holder by BastardKB x KarlK90")
   )
   (junction (at 195.58 107.95) (diameter 0) (color 0 0 0 0)
